File: transmissionLineTest.kicad_pcb (KiCad board)
At the start: 4 copper layers, 60 x 35 mm, 6 parts, among them J1 U.FL, J2 U.FL, J3 U.FL

Commit message: cleanup
Other:
- board size 60 x 35 mm -> 58.5 x 34 mm
Changed lines of the file:
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@@
     (effects (font (size 1.5 1.5) (thickness 0.3)))
   )
-  (gr_line (start 170 35) (end 110 35) (layer Edge.Cuts) (width 0.05))
-  (gr_line (start 170 70) (end 170 35) (layer Edge.Cuts) (width 0.05))
-  (gr_line (start 110 70) (end 170 70) (layer Edge.Cuts) (width 0.05))
-  (gr_line (start 110 35) (end 110 70) (layer Edge.Cuts) (width 0.05))
+  (gr_line (start 168.5 35) (end 110 35) (layer Edge.Cuts) (width 0.05))
+  (gr_line (start 168.5 69) (end 168.5 35) (layer Edge.Cuts) (width 0.05))
+  (gr_line (start 110 69) (end 168.5 69) (layer Edge.Cuts) (width 0.05))
+  (gr_line (start 110 35) (end 110 69) (layer Edge.Cuts) (width 0.05))
   (gr_text "33 Ohm" (at 122.555 38.735) (layer F.SilkS)
     (effects (font (size 1.5 1.5) (thickness 0.3)))
@@
     (polygon
       (pts
-        (xy 169.5 69.5) (xy 110.5 69.5) (xy 110.5 35.5) (xy 169.5 35.5)
+        (xy 168 68.5) (xy 110.5 68.5) (xy 110.5 35.5) (xy 168 35.5)
       )
     )

Commit message: add diff test
Parts:
- added J4: U.FL, Connector_Coaxial:U.FL_Hirose_U.FL-R-SMT-1_Vertical, B.Cu at (180.3, 46.4)
- added J5: U.FL, Connector_Coaxial:U.FL_Hirose_U.FL-R-SMT-1_Vertical, B.Cu at (180.3, 57.8)
- added JP6: Jumper_NO_Small, Jumper:SolderJumper-2_P1.3mm_Open_RoundedPad1.0x1.5mm, B.Cu at (113.0, 45.2)
- added JP7: Jumper_NO_Small, Jumper:SolderJumper-2_P1.3mm_Open_RoundedPad1.0x1.5mm, B.Cu at (113.0, 47.5)
- added JP8: Jumper_NO_Small, Jumper:SolderJumper-2_P1.3mm_Open_RoundedPad1.0x1.5mm, B.Cu at (113.0, 56.6)
- added JP9: Jumper_NO_Small, Jumper:SolderJumper-2_P1.3mm_Open_RoundedPad1.0x1.5mm, B.Cu at (113.0, 58.9)
- added TR1: ADT1-1WT+, RF_Mini-Circuits:Mini-Circuits_CD542_H2.84mm, B.Cu at (172.7, 46.4)
- added TR2: ADT1-1WT+, RF_Mini-Circuits:Mini-Circuits_CD542_H2.84mm, B.Cu at (172.7, 57.8)
- moved JP1 15.9 mm to (179.7, 40.6)
- moved JP2 15.9 mm to (179.7, 52.1)
- moved JP3 15.9 mm to (179.7, 63.5)
Connections:
- net Net-(J1-Pad1) renamed /33ohm
- net Net-(J2-Pad1) renamed /50ohm
- net Net-(J3-Pad1) renamed /75ohm
Routing:
- net /120ohm_P: track 0.00 -> 57.9 mm
- net /120ohm_N: track 0.00 -> 57.9 mm
- net /100ohm_P: track 0.00 -> 57.9 mm
- net /100ohm_N: track 0.00 -> 57.9 mm
- net /75ohm: track 47.8 -> 63.7 mm
- net /50ohm: track 47.8 -> 63.7 mm
- net /33ohm: track 47.8 -> 63.7 mm
- net Net-(J5-Pad1): track 0.00 -> 6.20 mm
- net Net-(J4-Pad1): track 0.00 -> 6.20 mm
- net GND: vias 75 -> 154
- added copper zone on B.Cu, net GND
- added copper zone on In2.Cu, net GND
Other:
- board size 58.5 x 34 mm -> 75 x 34 mm
- net class Diff 100ohm added: clearance 0.1524, trace_width 0.175006, via_dia 0.8, via_drill 0.4
- net class Diff 120ohm added: clearance 0.1524, trace_width 0.101092, via_dia 0.8, via_drill 0.4
- board text added: "100 Ohm"
- board text added: "120 Ohm"
